File: Project_Directory/on_board_pcb/on_board_pcb.kicad_sch (KiCad schematic)
At the start: 10 parts, among them U1 Teensy4.1

Commit message: preliminary pcb routing
Parts:
- U2: footprint Avionics_Footprints:BMP180 -> Avionics_Footprints:BMP388
Changed lines of the file:
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@@
 (kicad_sch
-	(version 20231120)
+	(version 20250114)
 	(generator "eeschema")
-	(generator_version "8.0")
+	(generator_version "9.0")
 	(paper "A4")
 	(junction
@@
 			)
 		)
-		(property "Footprint" "Avionics_Footprints:BMP180"
+		(property "Footprint" "Avionics_Footprints:BMP388"
 			(at 105.41 86.36 0)
 			(effects
@@
 		)
 	)
+	(embedded_fonts no)
 )

Commit message: p1 board semifinal
Parts:
- R1, R2, R3: footprint Resistor_THT:R_Axial_DIN0204_L3.6mm_D1.6mm_P1.90mm_Vertical -> Resistor_THT:R_Axial_DIN0207_L6.3mm_D2.5mm_P7.62mm_Horizontal
Connections:
- net GND1 is gone; now on net GND: U1.34 (GND), U3.1 (GND), U5.1 (GND)
- net GND: now also U1.1 (GND), U4.4 (GND)
- no-connect marks 60 -> 16
