File: Project_Directory/Avionics_Board_Rev_2/_autosave-Avionics_Board_Rev_2.kicad_sch (KiCad schematic)
At the start: 79 parts, among them J1 Battery, J10 PWM_1, J11 PWM_2, J12 PWM_3, J13 I2C, J14 UART, J15 Conn_Coaxial, J2 ARM, J3 PYRO_1, J4 PYRO_1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

Commit message: schematic changes
Parts:
- J1: footprint TerminalBlock_Phoenix:TerminalBlock_Phoenix_MKDS-1,5-2-5.08_1x02_P5.08mm_Horizontal -> Connector_AMASS:AMASS_XT60PW-M_1x02_P7.20mm_Horizontal
Connections:
- net +3.3V: now also U1.15 (3V3)
- net Buzzer: now also U1.33 (41_A17); no longer U1.16 (24_A10_TX6_SCL2)
- net CS_BMP: now also U1.26 (34_RX8); no longer U1.23 (31_CTX3)
- net CS_IMU: now also U1.27 (35_TX8); no longer U1.22 (30_CRX3)
- net GND: now also U1.1 (GND)
- net GPS_RX: now also U1.7 (5_IN2); no longer U1.42 (20_A6_TX5_LRCLK1)
- net GPS_TX: now also U1.6 (4_BCLK2); no longer U1.43 (21_A7_RX5_BCLK1)
- net GSM_RST: now also U1.25 (33_MCLK2); no longer U1.24 (32_OUT1B)
- net GSM_RX: now also U1.22 (30_CRX3); no longer U1.27 (35_TX8)
- net GSM_TX: now also U1.23 (31_CTX3); no longer U1.26 (34_RX8)
- net I2C1_SCL: now also U1.11 (9_OUT1C); no longer U1.38 (16_A2_RX4_SCL1)
- net I2C1_SDA: now also U1.10 (8_TX2_IN1); no longer U1.39 (17_A3_TX4_SDA1)
- net LED_B: now also U1.8 (6_OUT1D); no longer U1.41 (19_A5_SCL)
- net LED_G: now also U1.5 (3_LRCLK2); no longer U1.44 (22_A8_CTX1)
- net LED_R: now also U1.4 (2_OUT2); no longer U1.45 (23_A9_CRX1_MCLK1)
- net LoRa_CS: now also U1.43 (21_A7_RX5_BCLK1); no longer U1.6 (4_BCLK2)
- net LoRa_DIO1: now also U1.44 (22_A8_CTX1); no longer U1.5 (3_LRCLK2)
- net LoRa_INT: now also U1.45 (23_A9_CRX1_MCLK1); no longer U1.4 (2_OUT2)
- net LoRa_RST: now also U1.42 (20_A6_TX5_LRCLK1); no longer U1.7 (5_IN2)
- net PWM_1: now also U1.39 (17_A3_TX4_SDA1); no longer U1.17 (25_A11_RX6_SDA2)
- net PWM_2: now also U1.38 (16_A2_RX4_SCL1); no longer U1.20 (28_RX7)
- net PWM_3: now also U1.37 (15_A1_RX3_SPDIF_IN); no longer U1.21 (29_TX7)
- net PWM_4: now also U1.24 (32_OUT1B); no longer U1.25 (33_MCLK2)
- net PWM_5: now also U1.13 (11_MOSI_CTX1); no longer U1.28 (36_CS)
- net PWM_6: now also U1.12 (10_CS_MQSR); no longer U1.29 (37_CS)
- net PYRO_1_Trig: now also U1.29 (37_CS)
- net PYRO_1_continuity: now also U1.16 (24_A10_TX6_SCL2)
- net PYRO_2_Trig: now also U1.20 (28_RX7)
- net PYRO_2_continuity: now also U1.18 (26_A12_MOSI1)
- net PYRO_3_Trig: now also U1.28 (36_CS)
- net PYRO_3_continuity: now also U1.17 (25_A11_RX6_SDA2)
- net PYRO_4_Trig: now also U1.21 (29_TX7)
- net PYRO_4_continuity: now also U1.19 (27_A13_SCK1)
- net SPI0_MISO: now also U1.35 (13_SCK_LED); no longer U1.14 (12_MISO_MQSL)
- net SPI0_MOSI: now also U1.36 (14_A0_TX3_SPDIF_OUT); no longer U1.13 (11_MOSI_CTX1)
- net SPI0_SCK: now also U1.14 (12_MISO_MQSL); no longer U1.35 (13_SCK_LED)
- net SPI1_MISO: now also U1.46 (3V3); no longer U1.3 (1_TX1_CTX2_MISO1)
- net SPI1_MOSI: now also U1.31 (39_MISO1_OUT1A); no longer U1.18 (26_A12_MOSI1)
- net SPI1_SCK: now also U1.30 (38_CS1_IN1); no longer U1.19 (27_A13_SCK1)
- no-connect marks 0 -> 17
