File: Project_Directory/Avionics_Board_Rev_2/Avionics_Board_Rev_2.kicad_sch (KiCad schematic)
At the start: 79 parts, among them J1 Battery, J10 PWM_1, J11 PWM_2, J12 PWM_3, J13 I2C, J14 UART, J15 Conn_Coaxial, J2 ARM, J3 PYRO_1, J4 PYRO_1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

Commit message: schematic and pcb commit -1
Parts:
- added Q5: Drive_MOS, Package_TO_SOT_SMD:SC-59_Handsoldering, symbol Simulation_SPICE:NMOS
- C1: value IRFR024NPBF -> MOS_1
- C10: value IRFR024NPBF -> MOS_4
- C8: value IRFR024NPBF -> MOS_3
- C9: value IRFR024NPBF -> MOS_2
- J1: footprint TerminalBlock_Phoenix:TerminalBlock_Phoenix_MKDS-1,5-2-5.08_1x02_P5.08mm_Horizontal -> Connector_AMASS:AMASS_XT60PW-M_1x02_P7.20mm_Horizontal
- J4: value PYRO_1 -> PYRO_3
- J5: value PYRO_1 -> PYRO_2
- J6: value PYRO_1 -> PYRO_4
- renumbered Q2 to Q1, Q3 to Q2, Q1 to Q3
Connections:
- net SCL is gone; now on net I2C1_SCL: U4.10 (SCL)
- net SDA is gone; now on net I2C1_SDA: U4.9 (SDA)
- net +3.3V: now also JP1.3 (B), R22.1, U1.15 (3V3), U1.46 (3V3), U6.4 (GND); no longer JP1.1 (A), U6.1 (VCC)
- net +5V: now also JP1.1 (A), R26.1; no longer JP1.3 (B)
- net +BATT: now also J1.2 (Pin_2); no longer J1.1 (Pin_1)
- net ADSPU: no longer R22.1
- net BUCK_Out: now also U10.1 (VCC); no longer U10.2 (VCC)
- net Buzzer: now also U1.37 (15_A1_RX3_SPDIF_IN), Q5.2 (G); no longer R26.1, U1.16 (24_A10_TX6_SCL2)
- net CS_BMP: now also U1.28 (36_CS); no longer U1.23 (31_CTX3)
- net CS_IMU: now also U1.29 (37_CS); no longer U1.22 (30_CRX3)
- net GND: now also U1.1 (GND), U1.34 (GND), U1.47 (GND), U10.5 (GND), U6.1 (VCC), Q5.3 (S); no longer BZ1.2 (GND), U10.6 (GND), U6.4 (GND)
- net GPS_RX: now also U1.21 (29_TX7); no longer U1.42 (20_A6_TX5_LRCLK1)
- net GPS_TX: now also U1.20 (28_RX7); no longer U1.43 (21_A7_RX5_BCLK1)
- net GSM_RST: now also U1.25 (33_MCLK2), U10.4 (RST); no longer U1.24 (32_OUT1B), U10.3 (RST)
- net GSM_RX: now also U10.2 (RXT); no longer U10.4 (RXD)
- net GSM_TX: now also U10.3 (TXD); no longer U10.5 (TXD)
- net LED_B: now also U1.10 (8_TX2_IN1); no longer U1.41 (19_A5_SCL)
- net LED_G: now also U1.11 (9_OUT1C); no longer U1.44 (22_A8_CTX1)
- net LED_R: now also U1.12 (10_CS_MQSR); no longer U1.45 (23_A9_CRX1_MCLK1)
- net LoRa_CS: now also U1.24 (32_OUT1B); no longer U1.6 (4_BCLK2)
- net LoRa_DIO1: now also U1.32 (40_A16); no longer U1.5 (3_LRCLK2)
- net LoRa_INT: now also U1.36 (14_A0_TX3_SPDIF_OUT); no longer U1.4 (2_OUT2)
- net LoRa_RST: now also U1.33 (41_A17); no longer U1.7 (5_IN2)
- net PWM_1: now also U1.9 (7_RX2_OUT1A); no longer U1.17 (25_A11_RX6_SDA2)
- net PWM_2: now also U1.8 (6_OUT1D); no longer U1.20 (28_RX7)
- net PWM_3: now also U1.7 (5_IN2); no longer U1.21 (29_TX7)
- net PWM_4: now also U1.6 (4_BCLK2); no longer U1.25 (33_MCLK2)
- net PWM_5: now also U1.5 (3_LRCLK2); no longer U1.28 (36_CS)
- net PWM_6: now also U1.4 (2_OUT2); no longer U1.29 (37_CS)
- net PYRO_1_Trig: now also U1.3 (1_TX1_CTX2_MISO1)
- net PYRO_1_continuity: now also U1.40 (18_A4_SDA)
- net PYRO_2_Trig: now also U1.2 (0_RX1_CRX2_CS1)
- net PYRO_2_continuity: now also U1.41 (19_A5_SCL)
- net PYRO_3_Trig: now also U1.43 (21_A7_RX5_BCLK1)
- net PYRO_3_continuity: now also U1.42 (20_A6_TX5_LRCLK1)
- net PYRO_4_Trig: now also U1.45 (23_A9_CRX1_MCLK1)
- net PYRO_4_continuity: now also U1.44 (22_A8_CTX1)
- net SPI1_MISO: now also U1.31 (39_MISO1_OUT1A); no longer U1.3 (1_TX1_CTX2_MISO1)
- net Spare_I2C_SCL: now also U1.16 (24_A10_TX6_SCL2)
- net Spare_I2C_SDA: now also U1.17 (25_A11_RX6_SDA2)
- net Spare_UART_RX: now also U1.23 (31_CTX3)
- net Spare_UART_TX: now also U1.22 (30_CRX3)
- net at U4.4 (AIN0): now also U3.5 (Z); no longer U3.3 (X)
- net at U4.6 (AIN2): now also U3.3 (X); no longer U3.5 (Z)
- net D_3: now reaches C8.4, D3.2 (A), J4.1 (Pin_1), R9.1
- net GND_BATT: now reaches C7.4
- net GND_BATT: now also C1.3, C10.3, C8.3, C9.3, J1.1 (Pin_1); no longer J1.2 (Pin_2)
- net D_2: now reaches C9.4, D4.2 (A), J5.1 (Pin_1), R13.1
- net D_1: now reaches C1.4, D1.2 (A), J3.1 (Pin_1), R4.1
- net D_4: now reaches C10.4, D5.2 (A), J6.1 (Pin_1), R17.1
- net GNDPWR renamed GND_PWR
- net GND_PWR: no longer C1.3, C10.3, C8.3, C9.3
- new net: BZ1.2 (GND), Q5.1 (D)
- no-connect marks 0 -> 7
Other:
- moved on the sheet: BZ1, J13, J14, J2, R26, U1

Commit message: resistor values added
Parts:
- R1, R12, R16, R2, R8: value R -> 500k
- R10, R14, R18, R19, R20, R5: value R -> 10k
- R11, R13, R15, R17, R3, R4, R6, R7, R9: value R -> 20k
- R23, R24, R25: value R -> 100
Changed lines of the file:
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@@
 			)
 		)
-		(property "Value" "R"
+		(property "Value" "500k"
 			(at 132.588 195.072 0)
 			(effects
@@
 			)
 		)
-		(property "Value" "R"
+		(property "Value" "100"
 			(at 289.56 143.51 90)
 			(effects
@@
 			)
 		)
-		(property "Value" "R"
+		(property "Value" "20k"
 			(at 161.29 252.7299 0)
 			(effects
@@
 			)
 		)
-		(property "Value" "R"
+		(property "Value" "500k"
 			(at 31.75 146.0499 0)
 			(effects
@@
 			)
 		)
-		(property "Value" "R"
+		(property "Value" "100"
 			(at 289.306 138.43 90)
 			(effects
@@
 			)
 		)
-		(property "Value" "R"
+		(property "Value" "10k"
 			(at 161.29 264.1599 0)
 			(effects
@@
 			)
 		)
-		(property "Value" "R"
+		(property "Value" "500k"
 			(at 204.978 248.412 0)
 			(effects
@@
 			)
 		)
-		(property "Value" "R"
+		(property "Value" "10k"
 			(at 161.29 210.8199 0)
 			(effects
@@
 			)
 		)
-		(property "Value" "R"
+		(property "Value" "20k"
 			(at 125.73 199.8979 0)
 			(effects
@@
 			)
 		)
-		(property "Value" "R"
+		(property "Value" "20k"
 			(at 125.73 253.2379 0)
 			(effects
@@
 			)
 		)
-		(property "Value" "R"
+		(property "Value" "10k"
 			(at 21.59 31.7499 0)
 			(effects
@@
 			)
 		)
-		(property "Value" "R"
+		(property "Value" "10k"
 			(at 233.68 264.1599 0)
 			(effects
@@
 			)
 		)
-		(property "Value" "R"
+		(property "Value" "20k"
 			(at 161.29 199.3899 0)
 			(effects
@@
 			)
 		)
-		(property "Value" "R"
+		(property "Value" "500k"
 			(at 202.438 195.072 0)
 			(effects
@@
 			)
 		)
-		(property "Value" "R"
+		(property "Value" "20k"
 			(at 231.14 199.3899 0)
 			(effects
@@
 			)
 		)
-		(property "Value" "R"
+		(property "Value" "100"
 			(at 289.306 148.336 90)
 			(effects
@@
 			)
 		)
-		(property "Value" "R"
+		(property "Value" "500k"
 			(at 132.588 248.412 0)
 			(effects
@@
 			)
 		)
-		(property "Value" "R"
+		(property "Value" "10k"
 			(at 34.29 31.7499 0)
 			(effects
@@
 			)
 		)
-		(property "Value" "R"
+		(property "Value" "20k"
 			(at 36.83 168.9099 0)
 			(effects
@@
 			)
 		)
-		(property "Value" "R"
+		(property "Value" "20k"
 			(at 233.68 252.7299 0)
 			(effects
@@
 			)
 		)
-		(property "Value" "R"
+		(property "Value" "20k"
 			(at 198.12 253.2379 0)
 			(effects
@@
 			)
 		)
-		(property "Value" "R"
+		(property "Value" "20k"
 			(at 195.58 199.8979 0)
 			(effects
@@
 			)
 		)
-		(property "Value" "R"
+		(property "Value" "10k"
 			(at 231.14 210.8199 0)
 			(effects

Commit message: values changed 4/3/26
Parts:
- R10, R14, R18, R5: value 10k -> 100k
- R11, R15, R3, R7: value 20k -> 100k
- R13, R17, R4, R9: value 20k -> 300k
- R2: value 500k -> 100k
Changed lines of the file:
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@@
 			)
 		)
-		(property "Value" "20k"
+		(property "Value" "300k"
 			(at 161.29 252.7299 0)
 			(effects
@@
 			)
 		)
-		(property "Value" "500k"
+		(property "Value" "100k"
 			(at 31.75 146.0499 0)
 			(effects
@@
 			)
 		)
-		(property "Value" "10k"
+		(property "Value" "100k"
 			(at 161.29 264.1599 0)
 			(effects
@@
 			)
 		)
-		(property "Value" "10k"
+		(property "Value" "100k"
 			(at 161.29 210.8199 0)
 			(effects
@@
 			)
 		)
-		(property "Value" "20k"
+		(property "Value" "100k"
 			(at 125.73 199.8979 0)
 			(effects
@@
 			)
 		)
-		(property "Value" "20k"
+		(property "Value" "100k"
 			(at 125.73 253.2379 0)
 			(effects
@@
 			)
 		)
-		(property "Value" "10k"
+		(property "Value" "100k"
 			(at 233.68 264.1599 0)
 			(effects
@@
 			)
 		)
-		(property "Value" "20k"
+		(property "Value" "300k"
 			(at 161.29 199.3899 0)
 			(effects
@@
 			)
 		)
-		(property "Value" "20k"
+		(property "Value" "300k"
 			(at 231.14 199.3899 0)
 			(effects
@@
 			)
 		)
-		(property "Value" "20k"
+		(property "Value" "300k"
 			(at 233.68 252.7299 0)
 			(effects
@@
 			)
 		)
-		(property "Value" "20k"
+		(property "Value" "100k"
 			(at 198.12 253.2379 0)
 			(effects
@@
 			)
 		)
-		(property "Value" "20k"
+		(property "Value" "100k"
 			(at 195.58 199.8979 0)
 			(effects
@@
 			)
 		)
-		(property "Value" "10k"
+		(property "Value" "100k"
 			(at 231.14 210.8199 0)
 			(effects

Commit message: switch added 1
Parts:
- added J16: ON, TerminalBlock_Phoenix:TerminalBlock_Phoenix_MKDS-1,5-2-5.08_1x02_P5.08mm_Horizontal, symbol Connector:Conn_01x02_Pin
- added SW1: SW_DPDT_x2, Library:Switch exp, symbol Switch:SW_DPDT_x2
Connections:
- net +BATT: now also J16.2 (Pin_2), SW1.2 (B); no longer Buck_Converter1.5 (Vout), Buck_Converter1.6 (Vout), C4.1, U8.3 (VI)
- new net +BATT_C: Buck_Converter1.5 (Vout), Buck_Converter1.6 (Vout), C4.1, J16.1 (Pin_1), SW1.3 (C), U8.3 (VI)
Other:
- moved on the sheet: J2, R2

Commit message: corrected buckconverter and drive mos
Parts:
- Buck_Converter1: footprint VelR:buck converter -> VelR:buck converter_corrected
- Q1, Q2, Q3, Q4: footprint Package_TO_SOT_SMD:SC-59_Handsoldering -> Package_TO_SOT_SMD:SOT-23; symbol Simulation_SPICE:NMOS -> Transistor_FET:BSS138
Connections:
- net +BATT_C: now also Buck_Converter1.3 (Vin), Buck_Converter1.4 (Vin); no longer Buck_Converter1.5 (Vout), Buck_Converter1.6 (Vout)
- net BUCK_Out: now also Buck_Converter1.5 (Vout), Buck_Converter1.6 (Vout); no longer Buck_Converter1.3 (Vin), Buck_Converter1.4 (Vin)
- net GND: now also Buck_Converter1.7 (Vout), Buck_Converter1.8 (Vout), Q1.2 (S), Q2.2 (S), Q3.2 (S), Q4.2 (S); no longer Buck_Converter1.1 (Vin), Buck_Converter1.2 (Vin), Q1.3 (S), Q2.3 (S), Q3.3 (S), Q4.3 (S)
- net GND_PWR: now also Buck_Converter1.1 (Vin), Buck_Converter1.2 (Vin); no longer Buck_Converter1.7 (Vout), Buck_Converter1.8 (Vout)
- net PYRO_1_Trig: now also Q1.1 (G); no longer Q1.2 (G)
- net PYRO_2_Trig: now also Q2.1 (G); no longer Q2.2 (G)
- net PYRO_3_Trig: now also Q3.1 (G); no longer Q3.2 (G)
- net PYRO_4_Trig: now also Q4.1 (G); no longer Q4.2 (G)
- net at C1.1, R1.2: now also Q1.3 (D); no longer Q1.1 (D)
- net at C8.1, R8.2: now also Q3.3 (D); no longer Q3.1 (D)
- net at C10.1, R16.2: now also Q4.3 (D); no longer Q4.1 (D)
- net at C9.1, R12.2: now also Q2.3 (D); no longer Q2.1 (D)
Other:
- moved on the sheet: Buck_Converter1
Changed lines of the file:
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@@
 	(paper "A3")
 	(junction
+		(at 80.01 166.37)
+		(diameter 0)
+		(color 0 0 0 0)
+	)
+	(junction
 		(at 196.85 71.12)
 		(diameter 0)
@@
 	)
 	(junction
-		(at 140.97 240.03)
+		(at 54.61 176.53)
 		(diameter 0)
 		(color 0 0 0 0)
 	)
 	(junction
-		(at 41.91 182.88)
+		(at 140.97 240.03)
 		(diameter 0)
 		(color 0 0 0 0)
 	)
 	(junction
-		(at 158.75 193.04)
+		(at 41.91 182.88)
 		(diameter 0)
 		(color 0 0 0 0)
 	)
 	(junction
-		(at 54.61 163.83)
+		(at 158.75 193.04)
 		(diameter 0)
 		(color 0 0 0 0)
@@
 	)
 	(junction
-		(at 80.01 176.53)
-		(diameter 0)
-		(color 0 0 0 0)
-	)
-	(junction
 		(at 62.23 200.66)
 		(diameter 0)
@@
 	)
 	(junction
+		(at 80.01 176.53)
+		(diameter 0)
+		(color 0 0 0 0)
+	)
+	(junction
 		(at 137.16 199.39)
 		(diameter 0)
@@
 	)
 	(junction
-		(at 80.01 166.37)
+		(at 83.82 167.64)
 		(diameter 0)
 		(color 0 0 0 0)
 	)
 	(junction
-		(at 83.82 167.64)
+		(at 54.61 173.99)
 		(diameter 0)
 		(color 0 0 0 0)
@@
 	)
 	(junction
-		(at 54.61 176.53)
+		(at 146.05 242.57)
 		(diameter 0)
 		(color 0 0 0 0)
 	)
 	(junction
-		(at 146.05 242.57)
+		(at 25.4 163.83)
 		(diameter 0)
 		(color 0 0 0 0)
 	)
 	(junction
-		(at 25.4 163.83)
+		(at 34.29 163.83)
 		(diameter 0)
 		(color 0 0 0 0)
 	)
 	(junction
-		(at 34.29 163.83)
+		(at 54.61 163.83)
 		(diameter 0)
 		(color 0 0 0 0)
@@
 	(wire
 		(pts
+			(xy 54.61 162.56) (xy 54.61 163.83)
+		)
+		(stroke
+			(width 0)
+			(type default)
+		)
+	)
+	(wire
+		(pts
 			(xy 137.16 186.69) (xy 140.97 186.69)
 		)
@@
 	(wire
 		(pts
+			(xy 54.61 173.99) (xy 55.88 173.99)
+		)
+		(stroke
+			(width 0)
+			(type default)
+		)
+	)
+	(wire
+		(pts
 			(xy 25.4 128.27) (xy 26.67 128.27)
 		)
@@
 	(wire
 		(pts
-			(xy 54.61 162.56) (xy 54.61 163.83)
-		)
-		(stroke
-			(width 0)
-			(type default)
-		)
-	)
-	(wire
-		(pts
 			(xy 326.39 54.61) (xy 323.85 54.61)
 		)
@@
 	(wire
 		(pts
-			(xy 39.37 144.78) (xy 34.29 144.78)
+			(xy 54.61 163.83) (xy 54.61 166.37)
 		)
 		(stroke
@@
 	(wire
 		(pts
-			(xy 63.5 200.66) (xy 62.23 200.66)
+			(xy 39.37 144.78) (xy 34.29 144.78)
 		)
 		(stroke
@@
 	(wire
 		(pts
-			(xy 215.9 196.85) (xy 220.98 196.85)
+			(xy 63.5 200.66) (xy 62.23 200.66)
 		)
 		(stroke
@@
 	(wire
 		(pts
-			(xy 213.36 252.73) (xy 209.55 252.73)
+			(xy 215.9 196.85) (xy 220.98 196.85)
 		)
 		(stroke
@@
 	(wire
 		(pts
-			(xy 210.82 199.39) (xy 210.82 204.47)
+			(xy 213.36 252.73) (xy 209.55 252.73)
 		)
 		(stroke
@@
 	(wire
 		(pts
-			(xy 93.98 176.53) (xy 104.14 176.53)
+			(xy 210.82 199.39) (xy 210.82 204.47)
 		)
 		(stroke
@@
 	(wire
 		(pts
-			(xy 26.67 123.19) (xy 31.75 123.19)
+			(xy 93.98 176.53) (xy 104.14 176.53)
 		)
 		(stroke
@@
 	(wire
 		(pts
-			(xy 101.6 166.37) (xy 104.14 166.37)
+			(xy 26.67 123.19) (xy 31.75 123.19)
 		)
 		(stroke
@@
 	(wire
 		(pts
-			(xy 54.61 163.83) (xy 54.61 166.37)
+			(xy 101.6 166.37) (xy 104.14 166.37)
 		)
 		(stroke
@@
 	(symbol
 		(lib_id "VelR3:BUCK_CONVERTER_new")
-		(at 67.31 170.18 180)
+		(at 67.31 170.18 0)
+		(mirror x)
 		(unit 1)
 		(exclude_from_sim no)
@@
 		(on_board yes)
 		(dnp no)
-		(fields_autoplaced yes)
 		(property "Reference" "Buck_Converter1"
-			(at 67.31 154.94 0)
+			(at 67.31 185.42 0)
 			(effects
 				(font
@@
 		)
 		(property "Value" "buck converter"
-			(at 67.31 157.48 0)
+			(at 67.31 182.88 0)
 			(effects
 				(font
@@
 			)
 		)
-		(property "Footprint" "VelR:buck converter"
+		(property "Footprint" "VelR:buck converter_corrected"
 			(at 67.31 170.18 0)
 			(effects
@@
 	)
 	(symbol
-		(lib_id "Simulation_SPICE:NMOS")
+		(lib_id "Transistor_FET:BSS138")
 		(at 207.01 259.08 0)
 		(unit 1)
@@
 			)
 		)
-		(property "Footprint" "Package_TO_SOT_SMD:SC-59_Handsoldering"
-			(at 212.09 256.54 0)
+		(property "Footprint" "Package_TO_SOT_SMD:SOT-23"
+			(at 212.09 260.985 0)
 			(effects
 				(font
 					(size 1.27 1.27)
+					(italic yes)
 				)
+				(justify left)
 				(hide yes)
 			)
 		)
-		(property "Datasheet" "https://ngspice.sourceforge.io/docs/ngspice-html-manual/manual.xhtml#cha_MOSFETs"
-			(at 207.01 271.78 0)
+		(property "Datasheet" "https://www.onsemi.com/pub/Collateral/BSS138-D.PDF"
+			(at 212.09 262.89 0)
 			(effects
 				(font
 					(size 1.27 1.27)
 				)
+				(justify left)
 				(hide yes)
 			)
 		)
-		(property "Description" "N-MOSFET transistor, drain/source/gate"
+		(property "Description" "50V Vds, 0.22A Id, N-Channel MOSFET, SOT-23"
 			(at 207.01 259.08 0)
 			(effects
@@
 	)
 	(symbol
-		(lib_id "Simulation_SPICE:NMOS")
+		(lib_id "Transistor_FET:BSS138")
 		(at 134.62 205.74 0)
 		(unit 1)
@@
 			)
 		)
-		(property "Footprint" "Package_TO_SOT_SMD:SC-59_Handsoldering"
-			(at 139.7 203.2 0)
+		(property "Footprint" "Package_TO_SOT_SMD:SOT-23"
+			(at 139.7 207.645 0)
 			(effects
 				(font
 					(size 1.27 1.27)
+					(italic yes)
 				)
+				(justify left)
 				(hide yes)
 			)
 		)
-		(property "Datasheet" "https://ngspice.sourceforge.io/docs/ngspice-html-manual/manual.xhtml#cha_MOSFETs"
-			(at 134.62 218.44 0)
+		(property "Datasheet" "https://www.onsemi.com/pub/Collateral/BSS138-D.PDF"
+			(at 139.7 209.55 0)
 			(effects
 				(font
 					(size 1.27 1.27)
 				)
+				(justify left)
 				(hide yes)
 			)
 		)
-		(property "Description" "N-MOSFET transistor, drain/source/gate"
+		(property "Description" "50V Vds, 0.22A Id, N-Channel MOSFET, SOT-23"
 			(at 134.62 205.74 0)
 			(effects
@@
 	)
 	(symbol
-		(lib_id "Simulation_SPICE:NMOS")
+		(lib_id "Transistor_FET:BSS138")
 		(at 204.47 205.74 0)
 		(unit 1)
@@
 			)
 		)
-		(property "Footprint" "Package_TO_SOT_SMD:SC-59_Handsoldering"
-			(at 209.55 203.2 0)
+		(property "Footprint" "Package_TO_SOT_SMD:SOT-23"
+			(at 209.55 207.645 0)
 			(effects
 				(font
 					(size 1.27 1.27)
+					(italic yes)
 				)
+				(justify left)
 				(hide yes)
 			)
 		)
-		(property "Datasheet" "https://ngspice.sourceforge.io/docs/ngspice-html-manual/manual.xhtml#cha_MOSFETs"
-			(at 204.47 218.44 0)
+		(property "Datasheet" "https://www.onsemi.com/pub/Collateral/BSS138-D.PDF"
+			(at 209.55 209.55 0)
 			(effects
 				(font
 					(size 1.27 1.27)
 				)
+				(justify left)
 				(hide yes)
 			)
 		)
-		(property "Description" "N-MOSFET transistor, drain/source/gate"
+		(property "Description" "50V Vds, 0.22A Id, N-Channel MOSFET, SOT-23"
 			(at 204.47 205.74 0)
 			(effects
@@
 	)
 	(symbol
-		(lib_id "Simulation_SPICE:NMOS")
+		(lib_id "Transistor_FET:BSS138")
 		(at 134.62 259.08 0)
 		(unit 1)
@@
 			)
 		)
-		(property "Footprint" "Package_TO_SOT_SMD:SC-59_Handsoldering"
-			(at 139.7 256.54 0)
+		(property "Footprint" "Package_TO_SOT_SMD:SOT-23"
+			(at 139.7 260.985 0)
 			(effects
 				(font
 					(size 1.27 1.27)
+					(italic yes)
 				)
+				(justify left)
 				(hide yes)
 			)
 		)
-		(property "Datasheet" "https://ngspice.sourceforge.io/docs/ngspice-html-manual/manual.xhtml#cha_MOSFETs"
-			(at 134.62 271.78 0)
+		(property "Datasheet" "https://www.onsemi.com/pub/Collateral/BSS138-D.PDF"
+			(at 139.7 262.89 0)
 			(effects
 				(font
 					(size 1.27 1.27)
 				)
+				(justify left)
 				(hide yes)
 			)
 		)
-		(property "Description" "N-MOSFET transistor, drain/source/gate"
+		(property "Description" "50V Vds, 0.22A Id, N-Channel MOSFET, SOT-23"
 			(at 134.62 259.08 0)
 			(effects

Commit message: modification 1 7 mmarch
Parts:
- added H1, H2, H3, H4: MountingHole_Pad, MountingHole:MountingHole_3.2mm_M3_DIN965_Pad_TopBottom, symbol Mechanical:MountingHole_Pad
- Q5: footprint Package_TO_SOT_SMD:SC-59_Handsoldering -> Package_TO_SOT_SMD:SOT-23; symbol Simulation_SPICE:NMOS -> Transistor_FET:BSS84
Connections:
- net Buzzer: now also Q5.1 (G); no longer Q5.2 (G)
- net GND: now also Q5.2 (S), H1.1, H2.1, H3.1, H4.1; no longer Q5.3 (S)
- net PYRO_1_Trig: now also U1.2 (0_RX1_CRX2_CS1); no longer U1.3 (1_TX1_CTX2_MISO1)
- net PYRO_2_Trig: now also U1.3 (1_TX1_CTX2_MISO1); no longer U1.2 (0_RX1_CRX2_CS1)
- net at BZ1.2 (GND): now also Q5.3 (D); no longer Q5.1 (D)

Commit message: Modification 3 7th march
Parts:
- added R27, R28: 2.2k, Resistor_SMD:R_1206_3216Metric_Pad1.30x1.75mm_HandSolder, symbol Device:R
Connections:
- net +3.3V: now also R27.1, R28.2
- net Spare_I2C_SCL: now also R28.1
- net Spare_I2C_SDA: now also R27.2
