File: Project_Directory/Avionics_Board_Rev_2/Avionics_Board_Rev_2.kicad_pcb (KiCad board)
At the start: 2 copper layers, 60 x 120 mm, 64 parts, among them J1 Battery, J10 PWM_1, J11 PWM_2, J12 PWM_3, J13 I2C, J14 UART, J2 ARM, J3 PYRO_1, J4 PYRO_1, J5 PYRO_1, J6 PYRO_1, J7 PWM_4, J8 PWM_5, J9 PWM_6, Q1 Drive_MOS, Q2 Drive_MOS, Q3 Drive_MOS, Q4 Drive_MOS, U1 Teensy4.1, U10 GSM, U11 AP2127K-3.3, U2 LoRa - RFM95-W/PW, U5 AMS1117-3.3, U6 GPS, U7 GY-91, U8 AMS1117-5.0, U9 ADS1115 ADC

Commit message: temp
Parts:
- added REF**: AMASS_XT60IPW-M_1x03_P7.20mm_Horizontal, Connector_AMASS:AMASS_XT60IPW-M_1x03_P7.20mm_Horizontal, F.Cu at (150.7, 123.3)
- moved J1 29.0 mm to (162.2, 111.8)

Commit message: schematic and pcb commit -1
Parts:
- removed C6: ~, Capacitor_SMD:C_0603_1608Metric_Pad1.08x0.95mm_HandSolder
- removed the REF** at (150.7, 123.3)
- removed U9: ADS1115 ADC, Package_SO:TSSOP-10_3x3mm_P0.5mm
- added BZ1: Buzzer, VelR:Buzzer_TMB12A05, F.Cu at (136.5, 99.8)
- added C13: C, Capacitor_SMD:C_1206_3216Metric_Pad1.33x1.80mm_HandSolder, F.Cu at (142.7, 86.0)
- added C14: C, Capacitor_SMD:C_1210_3225Metric_Pad1.33x2.70mm_HandSolder, B.Cu at (132.9, 85.2)
- added J15: Conn_Coaxial, Connector_Coaxial:SMA_Samtec_SMA-J-P-H-ST-EM1_EdgeMount, B.Cu at (132.2, 27.4)
- added L1: L_Ferrite_Small, Inductor_SMD:L_1206_3216Metric_Pad1.22x1.90mm_HandSolder, F.Cu at (138.9, 84.7)
- added L2: L_Ferrite_Small, Inductor_SMD:L_1206_3216Metric_Pad1.22x1.90mm_HandSolder, F.Cu at (138.9, 87.2)
- added LED1: RGB, VelR:XL-z3535rgbasg_RGB_LED, F.Cu at (171.0, 84.0)
- added Q5: Drive_MOS, Package_TO_SOT_SMD:SC-59_Handsoldering, B.Cu at (139.7, 103.0)
- added R19: R, Capacitor_SMD:C_1206_3216Metric_Pad1.33x1.80mm_HandSolder, F.Cu at (139.2, 80.0)
- added R20: R, Capacitor_SMD:C_1206_3216Metric_Pad1.33x1.80mm_HandSolder, F.Cu at (139.2, 82.2)
- added R21: 10k, Capacitor_SMD:C_1206_3216Metric_Pad1.33x1.80mm_HandSolder, F.Cu at (132.9, 79.5)
- added R22: 10k, Capacitor_SMD:C_1206_3216Metric_Pad1.33x1.80mm_HandSolder, F.Cu at (130.4, 79.5)
- added R23: R, Resistor_SMD:R_1206_3216Metric_Pad1.30x1.75mm_HandSolder, F.Cu at (175.2, 76.8)
- added R24: R, Resistor_SMD:R_1206_3216Metric_Pad1.30x1.75mm_HandSolder, F.Cu at (172.5, 76.8)
- added R25: R, Resistor_SMD:R_1206_3216Metric_Pad1.30x1.75mm_HandSolder, F.Cu at (169.7, 76.8)
- added R26: R, Resistor_SMD:R_1206_3216Metric_Pad1.30x1.75mm_HandSolder, F.Cu at (141.9, 99.2)
- added REF**: MountingHole_3.2mm_M3_DIN965_Pad_TopBottom, MountingHole:MountingHole_3.2mm_M3_DIN965_Pad_TopBottom, F.Cu at (179.7, 35.7)
- added REF**: MountingHole_3.2mm_M3_DIN965_Pad_TopBottom, MountingHole:MountingHole_3.2mm_M3_DIN965_Pad_TopBottom, F.Cu at (179.7, 152.2)
- added REF**: MountingHole_3.2mm_M3_DIN965_Pad_TopBottom, MountingHole:MountingHole_3.2mm_M3_DIN965_Pad_TopBottom, F.Cu at (126.0, 152.2)
- added REF**: MountingHole_3.2mm_M3_DIN965_Pad_TopBottom, MountingHole:MountingHole_3.2mm_M3_DIN965_Pad_TopBottom, F.Cu at (126.0, 37.5)
- added U3: ADXL, VelR:ADXL377_SparkFun_Module, B.Cu at (128.0, 79.5)
- added U4: ADS1115IDGS, Package_SO:TSSOP-10_3x3mm_P0.5mm, F.Cu at (132.9, 85.0)
- C1: value IRFR024NPBF -> MOS_1; moved to B.Cu
- C10: value IRFR024NPBF -> MOS_4; moved to B.Cu
- C4, C5, R2, U8: moved to B.Cu
- C7, D2, U5: moved to F.Cu
- C8: value IRFR024NPBF -> MOS_3; moved to B.Cu
- C9: value IRFR024NPBF -> MOS_2; moved to B.Cu
- J1: footprint TerminalBlock_Phoenix:TerminalBlock_Phoenix_MKDS-1,5-2-5.08_1x02_P5.08mm_Horizontal -> Connector_AMASS:AMASS_XT60PW-M_1x02_P7.20mm_Horizontal
- J4: value PYRO_1 -> PYRO_3
- J5: value PYRO_1 -> PYRO_2
- J6: value PYRO_1 -> PYRO_4
- moved R2 125.9 mm to (149.4, 152.9)
- moved R9 124.7 mm to (170.7, 131.4), turned to 90 degrees
- moved R17 123.5 mm to (170.7, 141.4), turned to 90 degrees
- moved R8 123.5 mm to (169.4, 128.0), turned to 180 degrees
- moved R16 122.2 mm to (169.4, 137.7), turned to 180 degrees
- moved R10 121.0 mm to (168.4, 131.4), turned to -90 degrees
- moved C3 120.8 mm to (165.9, 144.9), turned to 180 degrees
- moved R15 119.8 mm to (163.2, 138.4)
- moved R18 119.7 mm to (168.4, 141.4), turned to -90 degrees
- moved C2 119.7 mm to (159.2, 147.8), turned to -90 degrees
- moved R1 119.2 mm to (169.2, 107.7), turned to 180 degrees
- moved R4 118.4 mm to (170.7, 111.5), turned to 90 degrees
- moved R5 115.2 mm to (168.4, 111.5), turned to -90 degrees
- moved R7 114.2 mm to (163.2, 128.7)
- moved R13 114.1 mm to (170.7, 121.5), turned to 90 degrees
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Connections:
- net Net-(D1-A) renamed /D_1
- net Net-(D3-A) renamed /D_3
- net Net-(D4-A) renamed /D_2
- net Net-(D5-A) renamed /D_4
- Buck_Converter1 pad 1: Net-(U11-GND) -> GND
- Buck_Converter1 pad 2: Net-(U11-GND) -> GND
- Buck_Converter1 pad 7: GNDPWR -> /GND_PWR
- Buck_Converter1 pad 8: GNDPWR -> /GND_PWR
- C1 pad 1: Net-(Q2-D) -> Net-(Q1-D)
- C1 pad 3: GNDPWR -> GND_BATT
- C10 pad 3: GNDPWR -> GND_BATT
- C11 pad 1: Net-(U11-GND) -> GND
- C12 pad 1: Net-(U11-GND) -> GND
- C7 pad 3: GNDPWR -> /GND_PWR
- C7 pad 4: Net-(J1-Pin_2) -> GND_BATT
- C8 pad 1: Net-(Q1-D) -> Net-(Q3-D)
- C8 pad 3: GNDPWR -> GND_BATT
- C9 pad 1: Net-(Q3-D) -> Net-(Q2-D)
- C9 pad 3: GNDPWR -> GND_BATT
- D2 pad 2: GNDPWR -> /GND_PWR
- J1 pad 1: +BATT -> GND_BATT
- J1 pad 2: Net-(J1-Pin_2) -> +BATT
- JP1 pad 1: +3.3V -> +5V
- JP1 pad 3: +5V -> +3.3V
- Q1 pad 2: /PYRO_3_Trig -> /PYRO_1_Trig
- Q2 pad 2: /PYRO_1_Trig -> /PYRO_2_Trig
- Q3 pad 2: /PYRO_2_Trig -> /PYRO_3_Trig
- R1 pad 2: Net-(Q2-D) -> Net-(Q1-D)
- R12 pad 2: Net-(Q3-D) -> Net-(Q2-D)
- R8 pad 2: Net-(Q1-D) -> Net-(Q3-D)
- U1 pad 1: unconnected-(U1-GND-Pad1) -> GND
- U1 pad 10: unconnected-(U1-8_TX2_IN1-Pad10) -> /LED_B
- U1 pad 11: unconnected-(U1-9_OUT1C-Pad11) -> /LED_G
- U1 pad 12: unconnected-(U1-10_CS_MQSR-Pad12) -> /LED_R
- U1 pad 15: unconnected-(U1-3V3-Pad15) -> +3.3V
- U1 pad 16: unconnected-(U1-24_A10_TX6_SCL2-Pad16) -> /Spare_I2C_SCL
- U1 pad 17: /PWM_1 -> /Spare_I2C_SDA
- U1 pad 2: unconnected-(U1-0_RX1_CRX2_CS1-Pad2) -> /PYRO_2_Trig
- U1 pad 20: /PWM_2 -> /GPS_TX
- U1 pad 21: /PWM_3 -> /GPS_RX
- U1 pad 22: /CS_IMU -> /Spare_UART_TX
- U1 pad 23: /CS_BMP -> /Spare_UART_RX
- U1 pad 24: /GSM_RST -> /LoRa_CS
- U1 pad 25: /PWM_4 -> /GSM_RST
- U1 pad 28: /PWM_5 -> /CS_BMP
- U1 pad 29: /PWM_6 -> /CS_IMU
- U1 pad 3: /SPI1_MISO -> /PYRO_1_Trig
- U1 pad 31: unconnected-(U1-39_MISO1_OUT1A-Pad31) -> /SPI1_MISO
- U1 pad 32: unconnected-(U1-40_A16-Pad32) -> /LoRa_DIO1
- U1 pad 33: unconnected-(U1-41_A17-Pad33) -> /LoRa_RST
- U1 pad 34: unconnected-(U1-GND-Pad34) -> GND
- U1 pad 36: unconnected-(U1-14_A0_TX3_SPDIF_OUT-Pad36) -> /LoRa_INT
- U1 pad 37: unconnected-(U1-15_A1_RX3_SPDIF_IN-Pad37) -> /Buzzer
- U1 pad 4: /LoRa_INT -> /PWM_6
- U1 pad 40: unconnected-(U1-18_A4_SDA-Pad40) -> /PYRO_1_continuity
- U1 pad 41: unconnected-(U1-19_A5_SCL-Pad41) -> /PYRO_2_continuity
- U1 pad 42: /GPS_RX -> /PYRO_3_continuity
- U1 pad 43: /GPS_TX -> /PYRO_3_Trig
- U1 pad 44: unconnected-(U1-22_A8_CTX1-Pad44) -> /PYRO_4_continuity
- U1 pad 45: unconnected-(U1-23_A9_CRX1_MCLK1-Pad45) -> /PYRO_4_Trig
- U1 pad 46: unconnected-(U1-3V3-Pad46) -> +3.3V
- U1 pad 47: unconnected-(U1-GND-Pad47) -> GND
- U1 pad 5: /LoRa_DIO1 -> /PWM_5
- U1 pad 58: unconnected-(U1-GND-Pad58) -> GND
- U1 pad 59: unconnected-(U1-GND-Pad59) -> GND
- U1 pad 6: /LoRa_CS -> /PWM_4
- U1 pad 7: /LoRa_RST -> /PWM_3
- U1 pad 8: unconnected-(U1-6_OUT1D-Pad8) -> /PWM_2
- U1 pad 9: unconnected-(U1-7_RX2_OUT1A-Pad9) -> /PWM_1
- U10 pad 1: (no net) -> /BUCK_Out
- U10 pad 2: /BUCK_Out -> /GSM_RX
- U10 pad 3: /GSM_RST -> /GSM_TX
- U10 pad 4: /GSM_RX -> /GSM_RST
- U10 pad 5: /GSM_TX -> GND
- U11 pad 2: Net-(U11-GND) -> GND
- U2 pad 9: Net-(J15-In) -> /LoRa_Antenna
- U6 pad 1: +3.3V -> GND
- U6 pad 4: GND -> +3.3V
Routing:
- net GND: track 0.00 -> 534.3 mm, vias 0 -> 8
- net +3.3V: track 0.00 -> 201.6 mm
- net /BUCK_Out: track 0.00 -> 148.7 mm, vias 0 -> 4
- net +5V: track 0.00 -> 129.8 mm, vias 0 -> 4
- net +VDC: track 0.00 -> 128.5 mm
- net +BATT: track 0.00 -> 96.2 mm
- net GND_BATT: track 0.00 -> 77.9 mm
- net /PYRO_4_continuity: track 0.00 -> 70.5 mm
- net /PYRO_3_continuity: track 0.00 -> 64.7 mm
- net /LoRa_CS: track 0.00 -> 64.5 mm, vias 0 -> 2
- net /PYRO_4_Trig: track 0.00 -> 63.3 mm
- net /PYRO_3_Trig: track 0.00 -> 57.9 mm
- net /PYRO_2_continuity: track 0.00 -> 57.1 mm
- net /PYRO_1_Trig: track 0.00 -> 54.2 mm
- net /PYRO_1_continuity: track 0.00 -> 49.6 mm
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Other:
- board size 60 x 120 mm -> 60 x 130 mm

Commit message: switch added 1
Parts:
- added J16: ON, TerminalBlock_Phoenix:TerminalBlock_Phoenix_MKDS-1,5-2-5.08_1x02_P5.08mm_Horizontal, F.Cu at (127.5, 111.7)
- added SW1: SW_DPDT_x2, Library:Switch exp, F.Cu at (123.2, 131.2)
- R1, R12, R16, R8: value R -> 500k
- R10, R11, R14, R15, R18, R2, R3, R5, R7: value R -> 100k
- R13, R17, R4, R9: value R -> 300k
- R19, R20: value R -> 10k
- R23, R24, R25: value R -> 100
- R6: value R -> 20k
- moved Buck_Converter1 10.0 mm to (141.9, 120.6)
- moved C4 1.77 mm to (153.2, 112.2)
- moved U8 1.61 mm to (153.2, 104.3)
- moved C5 0.90 mm to (153.7, 110.2)
- moved C12 0.83 mm to (145.6, 101.2)
Connections:
- Buck_Converter1 pad 5: +BATT -> +BATT_C
- Buck_Converter1 pad 6: +BATT -> +BATT_C
- C4 pad 1: +BATT -> +BATT_C
- U8 pad 3: +BATT -> +BATT_C
Routing:
- net +BATT_C: track 0.00 -> 61.0 mm
- net +BATT: track 96.2 -> 108.3 mm
- net /GND_PWR: track 21.8 -> 31.2 mm
- net GND: track 534.3 -> 539.1 mm

Commit message: switch update 2
Parts:
- moved J15 1.00 mm to (131.2, 27.4)
- moved U6 0.32 mm to (180.4, 48.2)
- moved R9 0.18 mm to (170.8, 131.6)
- moved R10 0.15 mm to (168.4, 131.6)
- moved Q3 0.10 mm to (164.3, 132.2)
Routing:
- net /PYRO_3_continuity: track 64.7 -> 28.4 mm
- net GND: track 539.1 -> 533.9 mm
- net /LoRa_Antenna: track 10.9 -> 11.6 mm
- added copper zone on B.Cu, net GND
- added copper zone on F.Cu, net GND

Commit message: Modification 1 on 5 march
Routing:
- net GND: track 533.9 -> 551.4 mm, vias 8 -> 16
- net /PYRO_2_Trig: track 33.6 -> 36.9 mm
- net /Spare_UART_RX: track 8.90 -> 10.4 mm
- net /SPI1_MISO: track 28.7 -> 29.5 mm
- removed copper zone on B.Cu, net GND

Commit message: Modification 2 5 march
Parts:
- C7, D2, R6: moved to B.Cu
- moved R6 9.55 mm to (131.0, 129.9), turned to -90 degrees
- moved J6 1.90 mm to (177.4, 144.1)
- moved D2 1.72 mm to (127.0, 135.2), turned to 0 degrees
- moved C7 1.65 mm to (126.8, 143.1)
- moved J3 0.90 mm to (177.4, 111.3)
- moved J4 0.90 mm to (177.4, 133.1)
- moved Q4 0.25 mm to (164.2, 142.2)
Routing:
- net GND: track 551.4 -> 559.8 mm, vias 16 -> 17
- net Net-(D2-K): track 5.53 -> 12.0 mm
- net /GND_PWR: track 31.2 -> 27.0 mm
- net /D_3: track 9.54 -> 11.8 mm
- net GND_BATT: track 77.9 -> 79.7 mm
- net /D_4: track 9.54 -> 11.2 mm
- net +BATT: track 108.3 -> 109.9 mm
- added copper zone on B.Cu, net GND
